Commit message: aruco gazebo

File: src/minik_gazebo/urdf/minik2.xacro (robot description, xacro)
@@ -1,8 +1,7 @@
 <?xml version="1.0" ?>
-<robot name="minik_gazebo2" xmlns:xacro="http://www.ros.org/wiki/xacro">
+<robot name="minik_gazebo" xmlns:xacro="http://www.ros.org/wiki/xacro">
   <xacro:include filename="$(find minik_gazebo)/urdf/materials.xacro" />
   <xacro:include filename="$(find minik_gazebo)/urdf/minik.gazebo" />
   <xacro:include filename="$(find minik_gazebo)/urdf/macros.xacro" />
-  <xacro:include filename="$(find minik_gazebo)/meshes/minik2.dae" />
   <link name="link_chassis">
     <!-- pose and inertial -->
@@ -80,6 +79,6 @@
        <xacro:cylinder_inertia mass="1" r="0.05" l="0.1" />
    </inertial>
-   <visual>
-       <origin xyz="0 0 0" rpy="0 0 0" />
+   <visual name="left_cam_visual">
+       <origin xyz="0 -0.05 0" rpy="0 1.57 0" />
        <geometry>
        <cylinder radius="0.05" length="0.1"/>
@@ -87,6 +86,19 @@
        <material name="white" />
    </visual>
-   <collision>
-       <origin xyz="0 0 0" rpy="0 0 0"/>
+   <collision name="left_cam_collision">
+       <origin xyz="0 -0.05 0" rpy="0 1.57 0"/>
+       <geometry>
+       <cylinder radius="0.05" length="0.1"/>
+       </geometry>
+   </collision>
+   <visual name="right_cam_visual">
+       <origin xyz="0 0.05 0" rpy="0 1.57 0" />
+       <geometry>
+       <cylinder radius="0.05" length="0.1"/>
+       </geometry>
+       <material name="white" />
+   </visual>
+   <collision name="right_cam_collision">
+       <origin xyz="0 0.05 0" rpy="0 1.57 0"/>
        <geometry>
        <cylinder radius="0.05" length="0.1"/>
@@ -95,5 +107,5 @@
    </link>
    <joint name="joint_sensor_laser" type="fixed">
-   <origin xyz="0.15 0 0.25" rpy="0 0 0"/>
+   <origin xyz="0.1 0 0.15" rpy="0 0 0"/>
    <parent link="link_chassis"/>
    <child link="sensor_laser"/>

File: src/minik_gazebo/urdf/minik3.xacro (robot description, xacro)
@@ -4,5 +4,4 @@
   <xacro:include filename="$(find minik_gazebo)/urdf/minik.gazebo" />
   <xacro:include filename="$(find minik_gazebo)/urdf/macros.xacro" />
-  <xacro:include filename="$(find minik_gazebo)/meshes/cube2.dae" />
   <link name="link_chassis">
     <!-- pose and inertial -->
@@ -22,5 +21,5 @@
       <origin rpy="0 0 0" xyz="0 0 -0.05"/>
       <geometry>
-        <mesh filename = "package://minik_gazebo/meshes/minik1.dae" scale="0.5 0.5 0.5"/>
+        <mesh filename = "package://minik_gazebo/meshes/minik3.dae" scale="0.5 0.5 0.5"/>
       </geometry>
       <!-- <material name="blue"/>-->
