Commit message: partial data realization

File: src/minik_gazebo/urdf/macros.xacro (robot description, xacro)
@@ -11,5 +11,5 @@
               <origin rpy="0 1.5707 1.5707" xyz="0 0 0"/>
               <geometry>
-                <cylinder length="0.04" radius="0.07"/>
+                <cylinder length="0.04" radius="0.06"/><!-- radius="0.07-->
               </geometry>
             </collision>
@@ -17,5 +17,5 @@
               <origin rpy="0 1.5707 1.5707" xyz="0 0 0"/>
               <geometry>
-                <cylinder length="0.04" radius="0.07"/>
+                <cylinder length="0.04" radius="0.06"/><!-- radius="0.07-->
               </geometry>
             </visual>

File: src/minik_gazebo/urdf/minik2.xacro (robot description, xacro)
@@ -8,12 +8,13 @@
     <pose>0 0 0.1 0 0 0</pose>
     <inertial>
-      <mass value="5"/>
-      <origin rpy="0 0 0" xyz="0 0 0.1"/>
+      <mass value="2"/>
+      <origin rpy="0 0 0" xyz="0 0 0"/>
       <inertia ixx="0.0395416666667" ixy="0" ixz="0" iyy="0.106208333333" iyz="0" izz="0.106208333333"/>
     </inertial>
     <!-- body -->
     <collision name="collision_chassis">
+      <origin rpy="0 0 0" xyz="0 0 -0.05"/>
       <geometry>
-        <box size="0.3 0.3 0.4"/>
+        <box size="0.3 0.3 0.3"/>
       </geometry>
     </collision>
@@ -25,7 +26,7 @@
       <!-- <material name="blue"/>-->
     </visual>
-    <!-- caster front -->
+    <!-- caster front-->
     <collision name="caster_front_collision">
-      <origin rpy=" 0 0 0" xyz="0.12 0 -0.22"/>
+      <origin rpy=" 0 0 0" xyz="0.13 0 -0.22"/>
       <geometry>
         <sphere radius="0.03"/>
@@ -43,12 +44,12 @@
     </collision>
     <visual name="caster_front_visual">
-      <origin rpy=" 0 0 0" xyz="0.12 0 -0.22"/>
+      <origin rpy=" 0 0 0" xyz="0.13 0 -0.22"/>
       <geometry>
         <sphere radius="0.03"/>
       </geometry>
     </visual>
-   <!-- caster back -->
+   <!-- caster back-->
     <collision name="caster_back_collision">
-      <origin rpy=" 0 0 0" xyz="-0.12 0 -0.22"/>
+      <origin rpy=" 0 0 0" xyz="-0.13 0 -0.22"/>
       <geometry>
         <sphere radius="0.03"/>
@@ -66,5 +67,5 @@
     </collision>
     <visual name="caster_back_visual">
-      <origin rpy=" 0 0 0" xyz="-0.12 0 -0.22"/>
+      <origin rpy=" 0 0 0" xyz="-0.13 0 -0.22"/>
       <geometry>
         <sphere radius="0.03"/>
@@ -77,5 +78,5 @@
        <origin xyz="0 0 0" rpy="0 0 0" />
        <mass value="1" />
-       <xacro:cylinder_inertia mass="1" r="0.05" l="0.1" />
+       <xacro:cylinder_inertia mass="0" r="0.05" l="0.1" />
    </inertial>
    <visual name="left_cam_visual">
@@ -111,7 +112,67 @@
    <child link="sensor_laser"/>
  </joint>
+ <!-- front caster
+   <link name="front_caster">
+     <pose>0 0 0 0 0 0</pose>
+     <inertial>
+       <mass value="1"/>
+       <origin rpy="0 0 0" xyz="0 0 0"/>
+       <inertia ixx="0" ixy="0" ixz="0" iyy="0" iyz="0" izz="0"/>
+     </inertial>
+    <visual name="front_caster_visual">
+        <origin xyz="0 0 0" rpy="0 0 0" />
+        <geometry>
+        <sphere radius="0.03"/>
+        </geometry>
+        <material name="white" />
+    </visual>
+    <collision name="front_caster_collision">
+      <origin xyz="0 0 0" rpy="0 0 0" />
+      <geometry>
+      <sphere radius="0.03"/>
+      </geometry>
+      <material name="white" />
+    </collision>
+    </link>
+    <joint name="joint_front_caster" type="planar">
+    <origin xyz="0.12 0 -0.22" rpy="0 0 0"/>
+    <parent link="link_chassis"/>
+    <child link="front_caster"/>
+    <axis rpy="0 0 0" xyz="0 0 1"/>
+    <joint_properties damping="0.0" friction="0.0"/>
+  </joint>-->
+  <!-- back caster
+    <link name="back_caster">
+      <pose>0 0 0 0 0 0</pose>
+      <inertial>
+        <mass value="1"/>
+        <origin rpy="0 0 0" xyz="0 0 0"/>
+        <inertia ixx="0" ixy="0" ixz="0" iyy="0" iyz="0" izz="0"/>
+      </inertial>
+     <visual name="back_caster_visual">
+         <origin xyz="0 0 0" rpy="0 0 0" />
+         <geometry>
+         <sphere radius="0.03"/>
+         </geometry>
+         <material name="white" />
+     </visual>
+     <collision name="back_caster_collision">
+       <origin xyz="0 0 0" rpy="0 0 0" />
+       <geometry>
+       <sphere radius="0.03"/>
+       </geometry>
+       <material name="white" />
+     </collision>
+     </link>
+     <joint name="joint_back_caster" type="planar">
+     <origin xyz="-0.12 0 -0.22" rpy="0 0 0"/>
+     <parent link="link_chassis"/>
+     <child link="back_caster"/>
+     <axis rpy="0 0 0" xyz="0 0 1"/>
+     <joint_properties damping="0.0" friction="0.0"/>
+   </joint>-->
   <xacro:link_wheel name="link_right_wheel" />
-  <xacro:joint_wheel name="joint_right_wheel" child="link_right_wheel" origin_xyz="0 -0.15 -0.18" />
+  <xacro:joint_wheel name="joint_right_wheel" child="link_right_wheel" origin_xyz="0 -0.2 -0.19" />
   <xacro:link_wheel name="link_left_wheel" />
-  <xacro:joint_wheel name="joint_left_wheel" child="link_left_wheel" origin_xyz="0 0.15 -0.18" />
+  <xacro:joint_wheel name="joint_left_wheel" child="link_left_wheel" origin_xyz="0 0.2 -0.19" />
 </robot>

File: src/minik_gazebo/urdf/minik2_2.xacro (robot description, xacro)
@@ -22,9 +22,9 @@
       <origin rpy="0 0 0" xyz="0 0 -0.05"/>
       <geometry>
-        <mesh filename = "package://minik_gazebo/meshes/minik4.dae" scale="0.5 0.5 0.5"/>
+        <mesh filename = "package://minik_gazebo/meshes/minik2.dae" scale="0.5 0.5 0.5"/>
       </geometry>
       <!-- <material name="blue"/>-->
     </visual>
-    <!-- caster front-->
+    <!-- caster front -->
     <collision name="caster_front_collision">
       <origin rpy=" 0 0 0" xyz="0.13 0 -0.22"/>
@@ -49,5 +49,5 @@
       </geometry>
     </visual>
-   <!-- caster back-->
+   <!-- caster back -->
     <collision name="caster_back_collision">
       <origin rpy=" 0 0 0" xyz="-0.13 0 -0.22"/>
@@ -78,5 +78,5 @@
        <origin xyz="0 0 0" rpy="0 0 0" />
        <mass value="1" />
-       <xacro:cylinder_inertia mass="0" r="0.05" l="0.1" />
+       <xacro:cylinder_inertia mass="1" r="0.05" l="0.1" />
    </inertial>
    <visual name="left_cam_visual">
@@ -112,64 +112,4 @@
    <child link="sensor_laser"/>
  </joint>
- <!-- front caster
-   <link name="front_caster">
-     <pose>0 0 0 0 0 0</pose>
-     <inertial>
-       <mass value="1"/>
-       <origin rpy="0 0 0" xyz="0 0 0"/>
-       <inertia ixx="0" ixy="0" ixz="0" iyy="0" iyz="0" izz="0"/>
-     </inertial>
-    <visual name="front_caster_visual">
-        <origin xyz="0 0 0" rpy="0 0 0" />
-        <geometry>
-        <sphere radius="0.03"/>
-        </geometry>
-        <material name="white" />
-    </visual>
-    <collision name="front_caster_collision">
-      <origin xyz="0 0 0" rpy="0 0 0" />
-      <geometry>
-      <sphere radius="0.03"/>
-      </geometry>
-      <material name="white" />
-    </collision>
-    </link>
-    <joint name="joint_front_caster" type="planar">
-    <origin xyz="0.12 0 -0.22" rpy="0 0 0"/>
-    <parent link="link_chassis"/>
-    <child link="front_caster"/>
-    <axis rpy="0 0 0" xyz="0 0 1"/>
-    <joint_properties damping="0.0" friction="0.0"/>
-  </joint>-->
-  <!-- back caster
-    <link name="back_caster">
-      <pose>0 0 0 0 0 0</pose>
-      <inertial>
-        <mass value="1"/>
-        <origin rpy="0 0 0" xyz="0 0 0"/>
-        <inertia ixx="0" ixy="0" ixz="0" iyy="0" iyz="0" izz="0"/>
-      </inertial>
-     <visual name="back_caster_visual">
-         <origin xyz="0 0 0" rpy="0 0 0" />
-         <geometry>
-         <sphere radius="0.03"/>
-         </geometry>
-         <material name="white" />
-     </visual>
-     <collision name="back_caster_collision">
-       <origin xyz="0 0 0" rpy="0 0 0" />
-       <geometry>
-       <sphere radius="0.03"/>
-       </geometry>
-       <material name="white" />
-     </collision>
-     </link>
-     <joint name="joint_back_caster" type="planar">
-     <origin xyz="-0.12 0 -0.22" rpy="0 0 0"/>
-     <parent link="link_chassis"/>
-     <child link="back_caster"/>
-     <axis rpy="0 0 0" xyz="0 0 1"/>
-     <joint_properties damping="0.0" friction="0.0"/>
-   </joint>-->
   <xacro:link_wheel name="link_right_wheel" />
   <xacro:joint_wheel name="joint_right_wheel" child="link_right_wheel" origin_xyz="0 -0.2 -0.19" />

File: src/minik_gazebo/urdf/minik3.xacro (robot description, xacro)
@@ -8,12 +8,13 @@
     <pose>0 0 0.1 0 0 0</pose>
     <inertial>
-      <mass value="5"/>
-      <origin rpy="0 0 0" xyz="0 0 0.1"/>
+      <mass value="2"/>
+      <origin rpy="0 0 0" xyz="0 0 0"/>
       <inertia ixx="0.0395416666667" ixy="0" ixz="0" iyy="0.106208333333" iyz="0" izz="0.106208333333"/>
     </inertial>
     <!-- body -->
     <collision name="collision_chassis">
+      <origin rpy="0 0 0" xyz="0 0 -0.05"/>
       <geometry>
-        <box size="0.3 0.3 0.4"/>
+        <box size="0.3 0.3 0.3"/>
       </geometry>
     </collision>
@@ -25,7 +26,7 @@
       <!-- <material name="blue"/>-->
     </visual>
-    <!-- caster front -->
+    <!-- caster front-->
     <collision name="caster_front_collision">
-      <origin rpy=" 0 0 0" xyz="0.12 0 -0.22"/>
+      <origin rpy=" 0 0 0" xyz="0.13 0 -0.22"/>
       <geometry>
         <sphere radius="0.03"/>
@@ -43,12 +44,12 @@
     </collision>
     <visual name="caster_front_visual">
-      <origin rpy=" 0 0 0" xyz="0.12 0 -0.22"/>
+      <origin rpy=" 0 0 0" xyz="0.13 0 -0.22"/>
       <geometry>
         <sphere radius="0.03"/>
       </geometry>
     </visual>
-   <!-- caster back -->
+   <!-- caster back-->
     <collision name="caster_back_collision">
-      <origin rpy=" 0 0 0" xyz="-0.12 0 -0.22"/>
+      <origin rpy=" 0 0 0" xyz="-0.13 0 -0.22"/>
       <geometry>
         <sphere radius="0.03"/>
@@ -66,5 +67,5 @@
     </collision>
     <visual name="caster_back_visual">
-      <origin rpy=" 0 0 0" xyz="-0.12 0 -0.22"/>
+      <origin rpy=" 0 0 0" xyz="-0.13 0 -0.22"/>
       <geometry>
         <sphere radius="0.03"/>
@@ -77,5 +78,5 @@
        <origin xyz="0 0 0" rpy="0 0 0" />
        <mass value="1" />
-       <xacro:cylinder_inertia mass="1" r="0.05" l="0.1" />
+       <xacro:cylinder_inertia mass="0" r="0.05" l="0.1" />
    </inertial>
    <visual name="left_cam_visual">
@@ -111,7 +112,67 @@
    <child link="sensor_laser"/>
  </joint>
+ <!-- front caster
+   <link name="front_caster">
+     <pose>0 0 0 0 0 0</pose>
+     <inertial>
+       <mass value="1"/>
+       <origin rpy="0 0 0" xyz="0 0 0"/>
+       <inertia ixx="0" ixy="0" ixz="0" iyy="0" iyz="0" izz="0"/>
+     </inertial>
+    <visual name="front_caster_visual">
+        <origin xyz="0 0 0" rpy="0 0 0" />
+        <geometry>
+        <sphere radius="0.03"/>
+        </geometry>
+        <material name="white" />
+    </visual>
+    <collision name="front_caster_collision">
+      <origin xyz="0 0 0" rpy="0 0 0" />
+      <geometry>
+      <sphere radius="0.03"/>
+      </geometry>
+      <material name="white" />
+    </collision>
+    </link>
+    <joint name="joint_front_caster" type="planar">
+    <origin xyz="0.12 0 -0.22" rpy="0 0 0"/>
+    <parent link="link_chassis"/>
+    <child link="front_caster"/>
+    <axis rpy="0 0 0" xyz="0 0 1"/>
+    <joint_properties damping="0.0" friction="0.0"/>
+  </joint>-->
+  <!-- back caster
+    <link name="back_caster">
+      <pose>0 0 0 0 0 0</pose>
+      <inertial>
+        <mass value="1"/>
+        <origin rpy="0 0 0" xyz="0 0 0"/>
+        <inertia ixx="0" ixy="0" ixz="0" iyy="0" iyz="0" izz="0"/>
+      </inertial>
+     <visual name="back_caster_visual">
+         <origin xyz="0 0 0" rpy="0 0 0" />
+         <geometry>
+         <sphere radius="0.03"/>
+         </geometry>
+         <material name="white" />
+     </visual>
+     <collision name="back_caster_collision">
+       <origin xyz="0 0 0" rpy="0 0 0" />
+       <geometry>
+       <sphere radius="0.03"/>
+       </geometry>
+       <material name="white" />
+     </collision>
+     </link>
+     <joint name="joint_back_caster" type="planar">
+     <origin xyz="-0.12 0 -0.22" rpy="0 0 0"/>
+     <parent link="link_chassis"/>
+     <child link="back_caster"/>
+     <axis rpy="0 0 0" xyz="0 0 1"/>
+     <joint_properties damping="0.0" friction="0.0"/>
+   </joint>-->
   <xacro:link_wheel name="link_right_wheel" />
-  <xacro:joint_wheel name="joint_right_wheel" child="link_right_wheel" origin_xyz="0 -0.15 -0.18" />
+  <xacro:joint_wheel name="joint_right_wheel" child="link_right_wheel" origin_xyz="0 -0.2 -0.19" />
   <xacro:link_wheel name="link_left_wheel" />
-  <xacro:joint_wheel name="joint_left_wheel" child="link_left_wheel" origin_xyz="0 0.15 -0.18" />
+  <xacro:joint_wheel name="joint_left_wheel" child="link_left_wheel" origin_xyz="0 0.2 -0.19" />
 </robot>

File: src/minik_gazebo/urdf/minik5.xacro (robot description, xacro)
@@ -8,12 +8,13 @@
     <pose>0 0 0.1 0 0 0</pose>
     <inertial>
-      <mass value="5"/>
-      <origin rpy="0 0 0" xyz="0 0 0.1"/>
+      <mass value="2"/>
+      <origin rpy="0 0 0" xyz="0 0 0"/>
       <inertia ixx="0.0395416666667" ixy="0" ixz="0" iyy="0.106208333333" iyz="0" izz="0.106208333333"/>
     </inertial>
     <!-- body -->
     <collision name="collision_chassis">
+      <origin rpy="0 0 0" xyz="0 0 -0.05"/>
       <geometry>
-        <box size="0.3 0.3 0.4"/>
+        <box size="0.3 0.3 0.3"/>
       </geometry>
     </collision>
@@ -25,7 +26,7 @@
       <!-- <material name="blue"/>-->
     </visual>
-    <!-- caster front -->
+    <!-- caster front-->
     <collision name="caster_front_collision">
-      <origin rpy=" 0 0 0" xyz="0.12 0 -0.22"/>
+      <origin rpy=" 0 0 0" xyz="0.13 0 -0.22"/>
       <geometry>
         <sphere radius="0.03"/>
@@ -43,12 +44,12 @@
     </collision>
     <visual name="caster_front_visual">
-      <origin rpy=" 0 0 0" xyz="0.12 0 -0.22"/>
+      <origin rpy=" 0 0 0" xyz="0.13 0 -0.22"/>
       <geometry>
         <sphere radius="0.03"/>
       </geometry>
     </visual>
-   <!-- caster back -->
+   <!-- caster back-->
     <collision name="caster_back_collision">
-      <origin rpy=" 0 0 0" xyz="-0.12 0 -0.22"/>
+      <origin rpy=" 0 0 0" xyz="-0.13 0 -0.22"/>
       <geometry>
         <sphere radius="0.03"/>
@@ -66,5 +67,5 @@
     </collision>
     <visual name="caster_back_visual">
-      <origin rpy=" 0 0 0" xyz="-0.12 0 -0.22"/>
+      <origin rpy=" 0 0 0" xyz="-0.13 0 -0.22"/>
       <geometry>
         <sphere radius="0.03"/>
@@ -77,5 +78,5 @@
        <origin xyz="0 0 0" rpy="0 0 0" />
        <mass value="1" />
-       <xacro:cylinder_inertia mass="1" r="0.05" l="0.1" />
+       <xacro:cylinder_inertia mass="0" r="0.05" l="0.1" />
    </inertial>
    <visual name="left_cam_visual">
@@ -111,7 +112,67 @@
    <child link="sensor_laser"/>
  </joint>
+ <!-- front caster
+   <link name="front_caster">
+     <pose>0 0 0 0 0 0</pose>
+     <inertial>
+       <mass value="1"/>
+       <origin rpy="0 0 0" xyz="0 0 0"/>
+       <inertia ixx="0" ixy="0" ixz="0" iyy="0" iyz="0" izz="0"/>
+     </inertial>
+    <visual name="front_caster_visual">
+        <origin xyz="0 0 0" rpy="0 0 0" />
+        <geometry>
+        <sphere radius="0.03"/>
+        </geometry>
+        <material name="white" />
+    </visual>
+    <collision name="front_caster_collision">
+      <origin xyz="0 0 0" rpy="0 0 0" />
+      <geometry>
+      <sphere radius="0.03"/>
+      </geometry>
+      <material name="white" />
+    </collision>
+    </link>
+    <joint name="joint_front_caster" type="planar">
+    <origin xyz="0.12 0 -0.22" rpy="0 0 0"/>
+    <parent link="link_chassis"/>
+    <child link="front_caster"/>
+    <axis rpy="0 0 0" xyz="0 0 1"/>
+    <joint_properties damping="0.0" friction="0.0"/>
+  </joint>-->
+  <!-- back caster
+    <link name="back_caster">
+      <pose>0 0 0 0 0 0</pose>
+      <inertial>
+        <mass value="1"/>
+        <origin rpy="0 0 0" xyz="0 0 0"/>
+        <inertia ixx="0" ixy="0" ixz="0" iyy="0" iyz="0" izz="0"/>
+      </inertial>
+     <visual name="back_caster_visual">
+         <origin xyz="0 0 0" rpy="0 0 0" />
+         <geometry>
+         <sphere radius="0.03"/>
+         </geometry>
+         <material name="white" />
+     </visual>
+     <collision name="back_caster_collision">
+       <origin xyz="0 0 0" rpy="0 0 0" />
+       <geometry>
+       <sphere radius="0.03"/>
+       </geometry>
+       <material name="white" />
+     </collision>
+     </link>
+     <joint name="joint_back_caster" type="planar">
+     <origin xyz="-0.12 0 -0.22" rpy="0 0 0"/>
+     <parent link="link_chassis"/>
+     <child link="back_caster"/>
+     <axis rpy="0 0 0" xyz="0 0 1"/>
+     <joint_properties damping="0.0" friction="0.0"/>
+   </joint>-->
   <xacro:link_wheel name="link_right_wheel" />
-  <xacro:joint_wheel name="joint_right_wheel" child="link_right_wheel" origin_xyz="0 -0.15 -0.18" />
+  <xacro:joint_wheel name="joint_right_wheel" child="link_right_wheel" origin_xyz="0 -0.2 -0.19" />
   <xacro:link_wheel name="link_left_wheel" />
-  <xacro:joint_wheel name="joint_left_wheel" child="link_left_wheel" origin_xyz="0 0.15 -0.18" />
+  <xacro:joint_wheel name="joint_left_wheel" child="link_left_wheel" origin_xyz="0 0.2 -0.19" />
 </robot>

File: src/minik_gazebo/urdf/minik5_2.xacro (robot description, xacro)
@@ -8,13 +8,12 @@
     <pose>0 0 0.1 0 0 0</pose>
     <inertial>
-      <mass value="2"/>
-      <origin rpy="0 0 0" xyz="0 0 0"/>
+      <mass value="5"/>
+      <origin rpy="0 0 0" xyz="0 0 0.1"/>
       <inertia ixx="0.0395416666667" ixy="0" ixz="0" iyy="0.106208333333" iyz="0" izz="0.106208333333"/>
     </inertial>
     <!-- body -->
     <collision name="collision_chassis">
-      <origin rpy="0 0 0" xyz="0 0 -0.05"/>
       <geometry>
-        <box size="0.3 0.3 0.3"/>
+        <box size="0.3 0.3 0.4"/>
       </geometry>
     </collision>
@@ -22,11 +21,11 @@
       <origin rpy="0 0 0" xyz="0 0 -0.05"/>
       <geometry>
-        <mesh filename = "package://minik_gazebo/meshes/minik4.dae" scale="0.5 0.5 0.5"/>
+        <mesh filename = "package://minik_gazebo/meshes/minik5.dae" scale="0.5 0.5 0.5"/>
       </geometry>
       <!-- <material name="blue"/>-->
     </visual>
-    <!-- caster front-->
+    <!-- caster front -->
     <collision name="caster_front_collision">
-      <origin rpy=" 0 0 0" xyz="0.13 0 -0.22"/>
+      <origin rpy=" 0 0 0" xyz="0.12 0 -0.22"/>
       <geometry>
         <sphere radius="0.03"/>
@@ -44,12 +43,12 @@
     </collision>
     <visual name="caster_front_visual">
-      <origin rpy=" 0 0 0" xyz="0.13 0 -0.22"/>
+      <origin rpy=" 0 0 0" xyz="0.12 0 -0.22"/>
       <geometry>
         <sphere radius="0.03"/>
       </geometry>
     </visual>
-   <!-- caster back-->
+   <!-- caster back -->
     <collision name="caster_back_collision">
-      <origin rpy=" 0 0 0" xyz="-0.13 0 -0.22"/>
+      <origin rpy=" 0 0 0" xyz="-0.12 0 -0.22"/>
       <geometry>
         <sphere radius="0.03"/>
@@ -67,5 +66,5 @@
     </collision>
     <visual name="caster_back_visual">
-      <origin rpy=" 0 0 0" xyz="-0.13 0 -0.22"/>
+      <origin rpy=" 0 0 0" xyz="-0.12 0 -0.22"/>
       <geometry>
         <sphere radius="0.03"/>
@@ -78,5 +77,5 @@
        <origin xyz="0 0 0" rpy="0 0 0" />
        <mass value="1" />
-       <xacro:cylinder_inertia mass="0" r="0.05" l="0.1" />
+       <xacro:cylinder_inertia mass="1" r="0.05" l="0.1" />
    </inertial>
    <visual name="left_cam_visual">
@@ -112,67 +111,7 @@
    <child link="sensor_laser"/>
  </joint>
- <!-- front caster
-   <link name="front_caster">
-     <pose>0 0 0 0 0 0</pose>
-     <inertial>
-       <mass value="1"/>
-       <origin rpy="0 0 0" xyz="0 0 0"/>
-       <inertia ixx="0" ixy="0" ixz="0" iyy="0" iyz="0" izz="0"/>
-     </inertial>
-    <visual name="front_caster_visual">
-        <origin xyz="0 0 0" rpy="0 0 0" />
-        <geometry>
-        <sphere radius="0.03"/>
-        </geometry>
-        <material name="white" />
-    </visual>
-    <collision name="front_caster_collision">
-      <origin xyz="0 0 0" rpy="0 0 0" />
-      <geometry>
-      <sphere radius="0.03"/>
-      </geometry>
-      <material name="white" />
-    </collision>
-    </link>
-    <joint name="joint_front_caster" type="planar">
-    <origin xyz="0.12 0 -0.22" rpy="0 0 0"/>
-    <parent link="link_chassis"/>
-    <child link="front_caster"/>
-    <axis rpy="0 0 0" xyz="0 0 1"/>
-    <joint_properties damping="0.0" friction="0.0"/>
-  </joint>-->
-  <!-- back caster
-    <link name="back_caster">
-      <pose>0 0 0 0 0 0</pose>
-      <inertial>
-        <mass value="1"/>
-        <origin rpy="0 0 0" xyz="0 0 0"/>
-        <inertia ixx="0" ixy="0" ixz="0" iyy="0" iyz="0" izz="0"/>
-      </inertial>
-     <visual name="back_caster_visual">
-         <origin xyz="0 0 0" rpy="0 0 0" />
-         <geometry>
-         <sphere radius="0.03"/>
-         </geometry>
-         <material name="white" />
-     </visual>
-     <collision name="back_caster_collision">
-       <origin xyz="0 0 0" rpy="0 0 0" />
-       <geometry>
-       <sphere radius="0.03"/>
-       </geometry>
-       <material name="white" />
-     </collision>
-     </link>
-     <joint name="joint_back_caster" type="planar">
-     <origin xyz="-0.12 0 -0.22" rpy="0 0 0"/>
-     <parent link="link_chassis"/>
-     <child link="back_caster"/>
-     <axis rpy="0 0 0" xyz="0 0 1"/>
-     <joint_properties damping="0.0" friction="0.0"/>
-   </joint>-->
   <xacro:link_wheel name="link_right_wheel" />
-  <xacro:joint_wheel name="joint_right_wheel" child="link_right_wheel" origin_xyz="0 -0.2 -0.19" />
+  <xacro:joint_wheel name="joint_right_wheel" child="link_right_wheel" origin_xyz="0 -0.15 -0.18" />
   <xacro:link_wheel name="link_left_wheel" />
-  <xacro:joint_wheel name="joint_left_wheel" child="link_left_wheel" origin_xyz="0 0.2 -0.19" />
+  <xacro:joint_wheel name="joint_left_wheel" child="link_left_wheel" origin_xyz="0 0.15 -0.18" />
 </robot>
