Commit message: last commit i hope so

File: src/minik_gazebo/urdf/minik1.xacro (robot description, xacro)
@@ -85,5 +85,5 @@
        <cylinder radius="0.05" length="0.1"/>
        </geometry>
-       <material name="white" />
+       <material name="blue" />
    </visual>
    <collision name="left_cam_collision">
@@ -98,5 +98,5 @@
        <cylinder radius="0.05" length="0.1"/>
        </geometry>
-       <material name="white" />
+       <material name="blue" />
    </visual>
    <collision name="right_cam_collision">

File: src/minik_gazebo/urdf/minik2.xacro (robot description, xacro)
@@ -85,5 +85,5 @@
        <cylinder radius="0.05" length="0.1"/>
        </geometry>
-       <material name="white" />
+       <material name="grey" />
    </visual>
    <collision name="left_cam_collision">
@@ -98,5 +98,5 @@
        <cylinder radius="0.05" length="0.1"/>
        </geometry>
-       <material name="white" />
+       <material name="grey" />
    </visual>
    <collision name="right_cam_collision">
